File: Project_Satellite.kicad_sch (KiCad schematic)
At the start: 64 parts, among them J1 Conn_01x02_Socket, J10 Conn_01x01_Socket, J11 Conn_01x01_Socket, J12 Conn_01x01_Socket, J15 Conn_01x01_Socket, J5 Conn_01x02_Socket, J6 Conn_01x02_Socket, J7 Conn_01x01_Socket, J8 Conn_01x02_Socket, J9 Conn_01x02_Socket, U3 TPS62933, U4 RASPBERRY_PI_ZERO_2_W, U5 TLV320AIC3254IRHBR, U6 MEMSMic, U7 MEMSMic, U8 TPA3118D2DAPR

Commit message: Laying out PCB components
Parts:
- added C1: 0.1uF, Capacitor_SMD:C_0805_2012Metric_Pad1.18x1.45mm_HandSolder, symbol Device:C
- J1, J5, J6, J8, J9: footprint Connector_PinHeader_2.54mm:PinHeader_1x02_P2.54mm_Horizontal -> Connector_PinHeader_2.54mm:PinHeader_1x02_P2.54mm_Vertical
- J10, J11, J12, J15, J7: footprint Connector_PinHeader_2.54mm:PinHeader_1x01_P2.54mm_Horizontal -> Connector_PinHeader_2.54mm:PinHeader_1x01_P2.54mm_Vertical
Connections:
- net +15V: now also C1.1
- net GND: now also C1.2
Other:
- moved on the sheet: C8, J15

Commit message: Initial placement and routing done. Need to fix DRC errors/warnings and create mic cutoff areas
Parts:
- added J13, J14, J16, J17, J18, J19, J2, J20, J21, J22, J23, J24, J3, J4: Conn_01x01_Socket, Connector_PinHeader_2.54mm:PinHeader_1x01_P2.54mm_Vertical, symbol Connector:Conn_01x01_Socket
Connections:
- net +3.3V: no longer J12.1 (Pin_1)
- net at C37.1, L4.2: now also J8.2 (Pin_2); no longer J9.1 (Pin_1)
- net at R7.1, U8.12 (MUTE): now also J12.1 (Pin_1)
- net at U4.11 (GPIO17/GPIO_GEN0): now also J19.1 (Pin_1)
- net at U4.13 (GPIO27/GPIO_GEN2): now also J24.1 (Pin_1)
- net at U4.15 (GPIO22/GPIO_GEN3): now also J20.1 (Pin_1)
- net at U4.16 (GPIO23/GPIO_GEN4): now also J21.1 (Pin_1)
- net at U4.18 (GPIO24/GPIO_GEN5): now also J22.1 (Pin_1)
- net at U4.24 (GPIO8/SPI_~{CE0}): now also J14.1 (Pin_1)
- net at U4.26 (GPIO7/SPI_~{CE1}): now also J13.1 (Pin_1)
- net at U4.29 (GPIO5): now also J3.1 (Pin_1)
- net at U4.31 (GPIO6): now also J4.1 (Pin_1)
- net at U4.32 (GPIO12): now also J16.1 (Pin_1)
- net at U4.33 (GPIO13): now also J17.1 (Pin_1)
- net at U4.36 (GPIO16): now also J18.1 (Pin_1)
- net at U4.37 (GPIO26): now also J23.1 (Pin_1)
- net at U4.7 (GPIO4/GPIO_GCLK): now also J2.1 (Pin_1)
- net at C36.2, L3.2: now also J9.1 (Pin_1); no longer J8.2 (Pin_2)
- no-connect marks 33 -> 19
Other:
- moved on the sheet: J12, J8, J9, R7

Commit message: Finished PCB design, do quick check and fabricate
Parts:
- added J25, J26, J27, J28: Conn_01x03_Socket, Connector_PinHeader_2.54mm:PinHeader_1x03_P2.54mm_Vertical, symbol Connector:Conn_01x03_Socket
Connections:
- net +3.3V: no longer C12.2, U4.1 (3V3_1)
- net GND: now also J25.3 (Pin_3), J26.3 (Pin_3); no longer U6.3 (GND), U6.4 (GND), U7.3 (GND), U7.4 (GND)
- net MICBIAS: now also J25.1 (Pin_1), J26.1 (Pin_1); no longer U6.2 (VDD), U7.2 (VDD)
- net at C18.2: now also J26.2 (Pin_2); no longer U7.1 (Out)
- net at U6.1 (Out): now also J27.2 (Pin_2); no longer C17.1
- new net: J27.1 (Pin_1), U6.2 (VDD)
- new net: J27.3 (Pin_3), U6.3 (GND), U6.4 (GND)
- new net: C17.1, J25.2 (Pin_2)
- new net: J28.2 (Pin_2), U7.1 (Out)
- new net: J28.1 (Pin_1), U7.2 (VDD)
- new net: J28.3 (Pin_3), U7.3 (GND), U7.4 (GND)
- new net +3V3: C12.2, U4.1 (3V3_1)
Other:
- moved on the sheet: U6, U7

Commit message: Final V1 commit
Other:
- moved on the sheet: J5
Changed lines of the file:
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@@
+	(wire
+		(pts
+			(xy 100.33 198.12) (xy 107.95 198.12)
+		)
+		(stroke
+			(width 0)
+			(type default)
+		)
+	)
 	(wire
 		(pts
@@
 	(wire
 		(pts
+			(xy 100.33 195.58) (xy 109.22 195.58)
+		)
+		(stroke
+			(width 0)
+			(type default)
+		)
+	)
+	(wire
+		(pts
 			(xy 256.54 130.81) (xy 256.54 151.13)
 		)
@@
 	(wire
 		(pts
+			(xy 109.22 195.58) (xy 109.22 201.93)
+		)
+		(stroke
+			(width 0)
+			(type default)
+		)
+	)
+	(wire
+		(pts
 			(xy 393.7 207.01) (xy 388.62 207.01)
 		)
@@
 	(wire
 		(pts
+			(xy 107.95 198.12) (xy 107.95 204.47)
+		)
+		(stroke
+			(width 0)
+			(type default)
+		)
+	)
+	(wire
+		(pts
 			(xy 445.77 165.1) (xy 445.77 168.91)
 		)
@@
 	(wire
 		(pts
+			(xy 107.95 204.47) (xy 110.49 204.47)
+		)
+		(stroke
+			(width 0)
+			(type default)
+		)
+	)
+	(wire
+		(pts
 			(xy 187.96 184.15) (xy 193.04 184.15)
+		)
+		(stroke
+			(width 0)
+			(type default)
+		)
+	)
+	(wire
+		(pts
+			(xy 109.22 201.93) (xy 110.49 201.93)
 		)
 		(stroke
@@
 			)
 			(justify left bottom)
-		)
-	)
-	(label "MICBIAS"
-		(at 273.05 255.27 180)
-		(effects
-			(font
-				(size 1.27 1.27)
-			)
-			(justify right bottom)
-		)
-	)
-	(label "MICBIAS"
-		(at 292.1 255.27 180)
-		(effects
-			(font
-				(size 1.27 1.27)
-			)
-			(justify right bottom)
 		)
 	)
@@
 	(symbol
 		(lib_id "Connector:Conn_01x02_Socket")
-		(at 105.41 204.47 180)
+		(at 95.25 198.12 180)
 		(unit 1)
 		(exclude_from_sim no)
@@
 		(fields_autoplaced yes)
 		(property "Reference" "J5"
-			(at 106.045 196.85 0)
+			(at 95.885 190.5 0)
 			(effects
 				(font
@@
 		)
 		(property "Value" "Conn_01x02_Socket"
-			(at 106.045 199.39 0)
+			(at 95.885 193.04 0)
 			(effects
 				(font
@@
 		)
 		(property "Footprint" "Connector_PinHeader_2.54mm:PinHeader_1x02_P2.54mm_Vertical"
-			(at 105.41 204.47 0)
+			(at 95.25 198.12 0)
 			(effects
 				(font
@@
 		)
 		(property "Datasheet" "~"
-			(at 105.41 204.47 0)
+			(at 95.25 198.12 0)
 			(effects
 				(font
@@
 		)
 		(property "Description" "Generic connector, single row, 01x02, script generated"
-			(at 105.41 204.47 0)
-			(effects
-				(font
+			(at 95.25 198.12 0)
+			(effects
+				(font
