File: Project_Satellite.kicad_sch (KiCad schematic)
At the start: 59 parts, among them J1 Conn_01x02_Socket, J25 Conn_01x03_Socket, J26 Conn_01x03_Socket, J27 Conn_01x03_Socket, J28 Conn_01x03_Socket, J8 Conn_01x02_Socket, J9 Conn_01x02_Socket, U3 TPS62933, U4 RASPBERRY_PI_ZERO_2_W, U5 TLV320AIC3254IRHBR, U6 MEMSMic, U7 MEMSMic, U8 TPA3118D2DAPR

Commit message: TPA3118 changes
Parts:
- removed C21, C22: 2.2uF, Capacitor_SMD:C_0603_1608Metric_Pad1.08x0.95mm_HandSolder, symbol Device:C
- removed C27, C29: 1uF, Capacitor_SMD:C_0603_1608Metric_Pad1.08x0.95mm_HandSolder, symbol Device:C
- removed C28: 0.1uF, Capacitor_SMD:C_0805_2012Metric_Pad1.18x1.45mm_HandSolder, symbol Device:C
- removed C30, C31, C32, C33: 220nF, Capacitor_SMD:C_0603_1608Metric_Pad1.08x0.95mm_HandSolder, symbol Device:C
- removed C35, C36, C37, C38: 680nF, Capacitor_SMD:C_0805_2012Metric_Pad1.18x1.45mm_HandSolder, symbol Device:C
- removed J27, J28: Conn_01x03_Socket, Connector_JST:JST_XH_B3B-XH-A_1x03_P2.50mm_Vertical, symbol Connector:Conn_01x03_Socket
- removed J8, J9: Conn_01x02_Socket, Connector_JST:JST_XH_B2B-XH-A_1x02_P2.50mm_Vertical, symbol Connector:Conn_01x02_Socket
- removed L2, L3, L4, L5: 10uH, Inductor_SMD:L_APV_APH0630, symbol Device:L
- removed R6: 5.6k, Resistor_SMD:R_0603_1608Metric_Pad0.98x0.95mm_HandSolder, symbol Device:R
- removed U6, U7: MEMSMic, MyFootprints:MEMSMic, symbol MySymbols:MEMSMic
- added C1: 0.1uF, Capacitor_SMD:C_0805_2012Metric_Pad1.18x1.45mm_HandSolder, symbol Device:C
- added C11, C4: 220uF, symbol Device:C
- added C2, C7: 1nF, symbol Device:C
- added C21, C22, C27, C28, C29: 1uF, symbol Device:C_Small
- added C3, C9: 100nF, symbol Device:C
- added C30, C31, C45, C46: 220nF, symbol Device:C_Small
- added C32, C33, C39, C40: 680nF, symbol Device:C_Small
- added C35, C36, C41, C42: 1nF, symbol Device:C_Small
- added C37, C38, C43, C44: 10nF, symbol Device:C_Small
- added J2, J3: Conn_01x02_Socket, symbol Connector:Conn_01x02_Socket
- added L2, L3, L4, L5: 10uH, symbol Device:L_Small
- added R10, R11, R12, R9: 3.3, symbol Device:R_Small
- added R5: 3.3, symbol Device:R
- added R6, R8: 100k, symbol Device:R_Small
- added R7: 20k, symbol Device:R_Small
- C19: value 2.2uF -> 100nF; footprint Capacitor_SMD:C_0603_1608Metric_Pad1.08x0.95mm_HandSolder -> (none)
- C20: value 2.2uF -> 10nF; footprint Capacitor_SMD:C_0603_1608Metric_Pad1.08x0.95mm_HandSolder -> (none)
- R3: value 50 -> 100k; footprint Resistor_SMD:R_0805_2012Metric_Pad1.20x1.40mm_HandSolder -> (none)
Connections:
- net +3V3 is gone; now on net +3.3V: C12.2, U4.1 (3V3_1)
- net +15V: now also C20.1, R3.1, C2.1, C3.1, C4.1, R5.1; no longer U8.17 (AVCC), U8.18 (PVCC), U8.19 (PVCC)
- net +5V: now also R2.2, C1.1; no longer R3.2
- net GND: now also C19.2, C20.2, C1.2, C11.2, C2.2, C22.1, C27.1, C29.1, C3.2, C32.1, C33.2, C35.2, C36.1, C37.2, C38.1, C39.2, C4.2, C40.1, C41.2, C42.1, C43.2, C44.1, C7.2, C9.2, R7.2, R8.2; no longer C19.1
- net MUTE: now also R8.1
- net SDZ: now also R3.2, U8.3 (FAULTZ)
- net at U8.6 (PLIMIT), U8.7 (GVDD): now also C27.2, R6.1
- net at U8.30 (BSPR): now also C30.1
- net at U8.29 (OUTPR): now also C30.2, L2.1
- net at U8.26 (BSNR): now also C31.1
- net at U8.27 (OUTNR): now also C31.2, L3.1
- net at U8.21 (OUTNL): now also C46.2, L5.1
- net at U8.20 (BSNL): now also C46.1
- net at U8.23 (OUTPL): now also C45.2, L4.1
- net at U8.11 (LINN): now also C29.2; no longer C19.2
- net at U5.22 (LOL): now also C28.1; no longer C20.1
- net at U5.23 (LOR): now also C21.1
- net at U8.4 (RINP): now also C21.2
- net at U8.10 (LINP): now also C28.2; no longer C20.2
- net at U8.8 (GAIN/SLV): now also R6.2, R7.1
- net at U8.24 (BSPL): now also C45.1
- net at U8.5 (RINN): now also C22.2
- net FAULTZ: no longer names the net of U4.16 (GPIO23/GPIO_GEN4)
- net FAULTZ: no longer U8.3 (FAULTZ)
- new net: C19.1, R5.2
- new net: C39.1, C41.1, L4.2, R11.1
- new net: C43.1, J3.1 (Pin_1), R11.2
- new net: C44.2, J3.2 (Pin_2), R12.2
- new net: C11.1, C7.1, C9.1, U8.17 (AVCC), U8.18 (PVCC), U8.19 (PVCC)
- new net: C32.2, C36.2, L3.2, R9.1
- new net: C37.1, J2.1 (Pin_1), R10.2
- new net: C33.1, C35.1, L2.2, R10.1
- new net: C40.2, C42.2, L5.2, R12.1
- new net: C38.2, J2.2 (Pin_2), R9.2
- no-connect marks 22 -> 32
Other:
- moved on the sheet: R1, R2

Commit message: Final V3 schematic
Parts:
- removed C1, C12: 0.1uF, Capacitor_SMD:C_0805_2012Metric_Pad1.18x1.45mm_HandSolder, symbol Device:C
- removed C16: 1uF, Capacitor_SMD:C_0603_1608Metric_Pad1.08x0.95mm_HandSolder, symbol Device:C
- removed D1: LED, LED_THT:LED_D3.0mm, symbol Device:LED
- removed R4: 220, Resistor_SMD:R_0805_2012Metric_Pad1.20x1.40mm_HandSolder, symbol Device:R
- added C16, C47: 0.1uF, symbol Device:C_Small
- added R13: 10k, symbol Device:R_Small
- added R14: 4.7k, symbol Device:R_Small
- added TP5, TP6: TestPoint, symbol Connector:TestPoint
- C13: value 1uF -> 10uF
- C15: value 0.1uF -> 10uF
- C26: value 0.1uF -> 1uF
Connections:
- net +3.3V: now also C16.2, C47.2, R14.2; no longer U4.1 (3V3_1), U4.17 (3V3_17), U5.30 (LDO_SELECT)
- net +5V: now also TP5.1; no longer U4.2 (5V_2), U4.4 (5V_4)
- net GND: now also R13.1, TP6.1; no longer U5.12 (SPI_SELECT)
- removed net MICBIAS: J25.1 (Pin_1), J26.1 (Pin_1), U5.19 (MICBIAS)
- new net: R13.2, U5.12 (SPI_SELECT)
- new net: C47.1, J25.1 (Pin_1)
- new net: R14.1, U5.30 (LDO_SELECT)
- new net: C16.1, J26.1 (Pin_1)
- no-connect marks 32 -> 37
Other:
- moved on the sheet: J25

Commit message: Fixed V2 schematic footprints
Parts:
- removed TP5, TP6: TestPoint, symbol Connector:TestPoint
- added J4: Conn_01x02_Socket, Connector_JST:JST_XH_B2B-XH-A_1x02_P2.50mm_Vertical, symbol Connector:Conn_01x02_Socket
- C10: footprint Capacitor_SMD:C_1206_3216Metric_Pad1.33x1.80mm_HandSolder -> Capacitor_THT:CP_Radial_D6.3mm_P2.50mm
- C11, C4: footprint (none) -> Capacitor_THT:CP_Radial_D8.0mm_P3.50mm
- C15: footprint Capacitor_SMD:C_0805_2012Metric_Pad1.18x1.45mm_HandSolder -> Capacitor_THT:CP_Radial_D5.0mm_P2.50mm
- C16, C32, C33, C39, C40, C47: footprint (none) -> Capacitor_SMD:C_0805_2012Metric_Pad1.18x1.45mm_HandSolder
- C19, C3, C9: value 100nF -> 0.1uF; footprint (none) -> Capacitor_SMD:C_0805_2012Metric_Pad1.18x1.45mm_HandSolder
- C2, C35, C36, C41, C42, C7: footprint (none) -> Capacitor_SMD:C_0402_1005Metric_Pad0.74x0.62mm_HandSolder
- C20, C21, C22, C27, C28, C29, C30, C31, C37, C38, C43, C44, C45, C46: footprint (none) -> Capacitor_SMD:C_0603_1608Metric_Pad1.08x0.95mm_HandSolder
- C8: footprint Capacitor_SMD:C_1206_3216Metric_Pad1.33x1.80mm_HandSolder -> Capacitor_THT:CP_Radial_D5.0mm_P2.50mm
- J2, J3: footprint (none) -> Connector_JST:JST_XH_B2B-XH-A_1x02_P2.50mm_Vertical
- L2, L3, L4, L5: footprint (none) -> Inductor_SMD:L_APV_APH0630
- R10, R11, R12, R13, R14, R3, R5, R6, R7, R8, R9: footprint (none) -> Resistor_THT:R_Axial_DIN0207_L6.3mm_D2.5mm_P5.08mm_Vertical
- TP1, TP2, TP3, TP4: footprint TestPoint:TestPoint_Pad_D1.0mm -> Connector_PinHeader_2.00mm:PinHeader_1x01_P2.00mm_Vertical
Connections:
- net +5V: now also J4.1 (Pin_1)
- net GND: now also J4.2 (Pin_2)
Other:
- moved on the sheet: R13

Commit message: V2 PCB Placement and Plane Placement
Parts:
- removed TP4: TestPoint, Connector_PinHeader_2.00mm:PinHeader_1x01_P2.00mm_Vertical, symbol Connector:TestPoint
- C13: footprint Capacitor_SMD:C_0603_1608Metric_Pad1.08x0.95mm_HandSolder -> Capacitor_THT:CP_Radial_D5.0mm_P2.50mm
Connections:
- net +3.3V: now also U4.1 (3V3_1), U4.17 (3V3_17)
- no-connect marks 37 -> 35
Changed lines of the file:
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@@
 	)
 	(junction
+		(at 173.99 195.58)
+		(diameter 0)
+		(color 0 0 0 0)
+	)
+	(junction
 		(at 179.07 255.27)
 		(diameter 0)
@@
 	)
 	(no_connect
-		(at 171.45 194.31)
-	)
-	(no_connect
 		(at 265.43 125.73)
 	)
@@
 	)
 	(no_connect
-		(at 171.45 196.85)
-	)
-	(no_connect
 		(at 339.09 203.2)
 	)
@@
 	(wire
 		(pts
+			(xy 171.45 194.31) (xy 173.99 194.31)
+		)
+		(stroke
+			(width 0)
+			(type default)
+		)
+	)
+	(wire
+		(pts
 			(xy 483.87 212.09) (xy 483.87 214.63)
 		)
@@
 	(wire
 		(pts
+			(xy 173.99 194.31) (xy 173.99 195.58)
+		)
+		(stroke
+			(width 0)
+			(type default)
+		)
+	)
+	(wire
+		(pts
+			(xy 173.99 196.85) (xy 171.45 196.85)
+		)
+		(stroke
+			(width 0)
+			(type default)
+		)
+	)
+	(wire
+		(pts
 			(xy 402.59 195.58) (xy 402.59 193.04)
 		)
@@
 	(wire
 		(pts
+			(xy 173.99 195.58) (xy 173.99 196.85)
+		)
+		(stroke
+			(width 0)
+			(type default)
+		)
+	)
+	(wire
+		(pts
 			(xy 389.89 222.25) (xy 387.35 222.25)
 		)
@@
 			)
 		)
-		(property "Footprint" "Capacitor_SMD:C_0603_1608Metric_Pad1.08x0.95mm_HandSolder"
+		(property "Footprint" "Capacitor_THT:CP_Radial_D5.0mm_P2.50mm"
 			(at 207.9752 228.6 0)
 			(effects
@@
 	)
 	(symbol
-		(lib_id "Connector:TestPoint")
-		(at 205.74 128.27 90)
-		(unit 1)
-		(exclude_from_sim no)
-		(in_bom yes)
-		(on_board yes)
-		(dnp no)
-		(property "Reference" "TP4"
-			(at 197.866 128.524 90)
-			(effects
-				(font
-					(size 1.27 1.27)
-				)
-			)
-		)
-		(property "Value" "TestPoint"
-			(at 198.628 130.556 90)
-			(effects
-				(font
-					(size 1.27 1.27)
-				)
-			)
-		)
-		(property "Footprint" "Connector_PinHeader_2.00mm:PinHeader_1x01_P2.00mm_Vertical"
-			(at 205.74 123.19 0)
-			(effects
-				(font
-					(size 1.27 1.27)
-				)
-				(hide yes)
-			)
-		)
-		(property "Datasheet" "~"
-			(at 205.74 123.19 0)
-			(effects
-				(font
-					(size 1.27 1.27)
-				)
-				(hide yes)
-			)
-		)
-		(property "Description" "test point"
-			(at 205.74 128.27 0)
-			(effects
-				(font
-					(size 1.27 1.27)
-				)
-				(hide yes)
-			)
-		)
-		(pin "1"
-		)
-		(instances
-			(project "Project_Satellite"
-				(path "/09bbc44e-8029-468d-a6fc-2a31dfd55e08"
-					(reference "TP4")
-					(unit 1)
-				)
-			)
-		)
-	)
-	(symbol
 		(lib_id "Device:L")
 		(at 304.8 123.19 90)
@@
 					(unit 1)
 				)
+			)
+		)
+	)
+	(symbol
+		(lib_id "power:+3.3V")
+		(at 173.99 195.58 270)
+		(unit 1)
+		(exclude_from_sim no)
+		(in_bom yes)
+		(on_board yes)
+		(dnp no)
+		(fields_autoplaced yes)
+		(property "Reference" "#PWR021"
+			(at 170.18 195.58 0)
+			(effects
+				(font
+					(size 1.27 1.27)
+				)
+				(hide yes)
+			)
+		)
+		(property "Value" "+3.3V"
+			(at 177.8 195.5799 90)
+			(effects
+				(font
+					(size 1.27 1.27)
+				)
+				(justify left)
+			)
+		)
+		(property "Footprint" ""
+			(at 173.99 195.58 0)
+			(effects
+				(font
+					(size 1.27 1.27)
+				)
+				(hide yes)
+			)
+		)
+		(property "Datasheet" ""
+			(at 173.99 195.58 0)
+			(effects
+				(font
+					(size 1.27 1.27)
+				)
+				(hide yes)
+			)
+		)
+		(property "Description" "Power symbol creates a global label with name \"+3.3V\""
+			(at 173.99 195.58 0)
+			(effects
+				(font
+					(size 1.27 1.27)
+				)
+				(hide yes)
+			)
+		)
+		(pin "1"
+		)
+		(instances
+			(project ""
+				(path "/09bbc44e-8029-468d-a6fc-2a31dfd55e08"
+					(reference "#PWR021")
+					(unit 1)
+				)

Commit message: Fully routed PCB V2 with Mic boards
Parts:
- J1: footprint Connector_JST:JST_XH_B2B-XH-A_1x02_P2.50mm_Vertical -> Connector_PinHeader_2.54mm:PinHeader_1x02_P2.54mm_Vertical
Connections:
- net MUTE: now also U4.36 (GPIO16); no longer U4.15 (GPIO22/GPIO_GEN3)
- net RESET: now also U4.11 (GPIO17/GPIO_GEN0); no longer U4.36 (GPIO16)
- net SDZ: now also U4.15 (GPIO22/GPIO_GEN3); no longer U4.11 (GPIO17/GPIO_GEN0)
Changed lines of the file:
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@@
 		)
 	)
-	(label "SDZ"
+	(label "RESET"
 		(at 171.45 207.01 0)
 		(effects
@@
 		)
 	)
-	(label "MUTE"
+	(label "SDZ"
 		(at 171.45 219.71 0)
 		(effects
@@
 		)
 	)
-	(label "RESET"
+	(label "MUTE"
 		(at 171.45 204.47 0)
 		(effects
@@
 			)
 		)
-		(property "Footprint" "Connector_JST:JST_XH_B2B-XH-A_1x02_P2.50mm_Vertical"
+		(property "Footprint" "Connector_PinHeader_2.54mm:PinHeader_1x02_P2.54mm_Vertical"
 			(at 200.66 125.73 0)
 			(effects
@@
 		(on_board yes)
 		(dnp no)
-		(fields_autoplaced yes)
 		(property "Reference" "R14"
 			(at 353.06 171.45 90)
