File: _autosave-Project_Satellite.kicad_sch (KiCad schematic)
At the start: 59 parts, among them J1 Conn_01x02_Socket, J25 Conn_01x03_Socket, J26 Conn_01x03_Socket, J27 Conn_01x03_Socket, J28 Conn_01x03_Socket, J8 Conn_01x02_Socket, J9 Conn_01x02_Socket, U3 TPS62933, U4 RASPBERRY_PI_ZERO_2_W, U5 TLV320AIC3254IRHBR, U6 MEMSMic, U7 MEMSMic, U8 TPA3118D2DAPR

Commit message: started laying out v2 pcb design
Parts:
- removed R3: 50, Resistor_SMD:R_0805_2012Metric_Pad1.20x1.40mm_HandSolder, symbol Device:R
- added TP5: TestPoint, TestPoint:TestPoint_Pad_D1.0mm, symbol Connector:TestPoint
Connections:
- net +15V: now also TP5.1
- net +5V: now also R2.2
Other:
- moved on the sheet: R1, R2
Changed lines of the file:
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@@
 	)
 	(junction
-		(at 289.56 138.43)
-		(diameter 0)
-		(color 0 0 0 0)
-	)
-	(junction
 		(at 294.64 284.48)
 		(diameter 0)
@@
 	)
 	(junction
+		(at 220.98 123.19)
+		(diameter 0)
+		(color 0 0 0 0)
+	)
+	(junction
 		(at 179.07 257.81)
 		(diameter 0)
@@
 	)
 	(junction
+		(at 289.56 140.97)
+		(diameter 0)
+		(color 0 0 0 0)
+	)
+	(junction
 		(at 207.01 220.98)
 		(diameter 0)
@@
 	(wire
 		(pts
+			(xy 289.56 143.51) (xy 289.56 140.97)
+		)
+		(stroke
+			(width 0)
+			(type default)
+		)
+	)
+	(wire
+		(pts
 			(xy 292.1 264.16) (xy 292.1 266.7)
 		)
@@
 	(wire
 		(pts
-			(xy 353.06 123.19) (xy 353.06 146.05)
+			(xy 353.06 123.19) (xy 353.06 140.97)
 		)
 		(stroke
@@
 	(wire
 		(pts
-			(xy 313.69 138.43) (xy 313.69 146.05)
-		)
-		(stroke
-			(width 0)
-			(type default)
-		)
-	)
-	(wire
-		(pts
 			(xy 241.3 228.6) (xy 241.3 234.95)
 		)
@@
 	(wire
 		(pts
-			(xy 215.9 123.19) (xy 223.52 123.19)
+			(xy 215.9 123.19) (xy 220.98 123.19)
 		)
 		(stroke
@@
 	(wire
 		(pts
-			(xy 309.88 138.43) (xy 313.69 138.43)
+			(xy 309.88 140.97) (xy 353.06 140.97)
 		)
 		(stroke
@@
 	(wire
 		(pts
+			(xy 289.56 140.97) (xy 289.56 138.43)
+		)
+		(stroke
+			(width 0)
+			(type default)
+		)
+	)
+	(wire
+		(pts
 			(xy 171.45 214.63) (xy 214.63 214.63)
 		)
@@
 	(wire
 		(pts
-			(xy 327.66 146.05) (xy 353.06 146.05)
-		)
-		(stroke
-			(width 0)
-			(type default)
-		)
-	)
-	(wire
-		(pts
 			(xy 171.45 260.35) (xy 179.07 260.35)
 		)
@@
 	(wire
 		(pts
-			(xy 289.56 138.43) (xy 302.26 138.43)
+			(xy 289.56 140.97) (xy 302.26 140.97)
 		)
 		(stroke
@@
 	(wire
 		(pts
+			(xy 220.98 123.19) (xy 223.52 123.19)
+		)
+		(stroke
+			(width 0)
+			(type default)
+		)
+	)
+	(wire
+		(pts
 			(xy 394.97 173.99) (xy 394.97 184.15)
 		)
@@
 	(wire
 		(pts
-			(xy 313.69 146.05) (xy 320.04 146.05)
-		)
-		(stroke
-			(width 0)
-			(type default)
-		)
-	)
-	(wire
-		(pts
 			(xy 273.05 266.7) (xy 269.24 266.7)
 		)
@@
 	(symbol
 		(lib_id "Device:R")
-		(at 306.07 138.43 90)
+		(at 306.07 140.97 90)
 		(unit 1)
 		(exclude_from_sim no)
@@
 		(fields_autoplaced yes)
 		(property "Reference" "R2"
-			(at 306.07 132.08 90)
+			(at 306.07 134.62 90)
 			(effects
 				(font
@@
 		)
 		(property "Value" "53.6k"
-			(at 306.07 134.62 90)
+			(at 306.07 137.16 90)
 			(effects
 				(font
@@
 		)
 		(property "Footprint" "Resistor_SMD:R_0603_1608Metric_Pad0.98x0.95mm_HandSolder"
-			(at 306.07 140.208 90)
+			(at 306.07 142.748 90)
 			(effects
 				(font
@@
 		)
 		(property "Datasheet" "~"
-			(at 306.07 138.43 0)
+			(at 306.07 140.97 0)
 			(effects
 				(font
@@
 		)
 		(property "Description" "Resistor"
-			(at 306.07 138.43 0)
+			(at 306.07 140.97 0)
 			(effects
 				(font
@@
 	(symbol
 		(lib_id "power:GND")
-		(at 289.56 146.05 0)
+		(at 289.56 151.13 0)
 		(unit 1)
 		(exclude_from_sim no)
@@
 		(fields_autoplaced yes)
 		(property "Reference" "#PWR017"
-			(at 289.56 152.4 0)
+			(at 289.56 157.48 0)
 			(effects
 				(font
@@
 		)
 		(property "Value" "GND"
-			(at 289.56 151.13 0)
+			(at 289.56 156.21 0)
 			(effects
 				(font
@@
 		)
 		(property "Footprint" ""
-			(at 289.56 146.05 0)
+			(at 289.56 151.13 0)
 			(effects
 				(font
@@
 		)
 		(property "Datasheet" ""
-			(at 289.56 146.05 0)
+			(at 289.56 151.13 0)
 			(effects
 				(font
@@
 		)
 		(property "Description" "Power symbol creates a global label with name \"GND\" , ground"
-			(at 289.56 146.05 0)
+			(at 289.56 151.13 0)
 			(effects
 				(font
@@
 	)
 	(symbol
+		(lib_id "Connector:TestPoint")
+		(at 220.98 123.19 0)
+		(unit 1)
+		(exclude_from_sim no)
+		(in_bom yes)
+		(on_board yes)
+		(dnp no)
+		(property "Reference" "TP5"
+			(at 221.488 115.062 0)
+			(effects
+				(font
+					(size 1.27 1.27)
+				)
+				(justify left)
+			)
+		)
+		(property "Value" "TestPoint"
+			(at 219.202 117.602 0)
+			(effects
+				(font
+					(size 1.27 1.27)
+				)
+				(justify left)
+			)
+		)
+		(property "Footprint" "TestPoint:TestPoint_Pad_D1.0mm"
+			(at 226.06 123.19 0)
+			(effects
+				(font
+					(size 1.27 1.27)
+				)
+				(hide yes)
+			)
+		)
+		(property "Datasheet" "~"
+			(at 226.06 123.19 0)
+			(effects
+				(font
+					(size 1.27 1.27)
+				)
+				(hide yes)
+			)
+		)
+		(property "Description" "test point"
+			(at 220.98 123.19 0)
+			(effects
+				(font
+					(size 1.27 1.27)
+				)
+				(hide yes)
+			)
+		)
+		(pin "1"
+		)
+		(instances
+			(project "Project_Satellite"
+				(path "/09bbc44e-8029-468d-a6fc-2a31dfd55e08"
+					(reference "TP5")
+					(unit 1)
+				)
+			)
+		)
+	)
+	(symbol
 		(lib_id "Device:C")
 		(at 514.35 167.64 0)
@@
 	(symbol
 		(lib_id "Device:R")
-		(at 289.56 142.24 0)
+		(at 289.56 147.32 0)
 		(unit 1)
 		(exclude_from_sim no)
@@
 		(fields_autoplaced yes)
 		(property "Reference" "R1"
-			(at 292.1 140.9699 0)
+			(at 292.1 146.0499 0)
 			(effects
 				(font
@@
 		)
 		(property "Value" "10.2k"
-			(at 292.1 143.5099 0)
+			(at 292.1 148.5899 0)
 			(effects
 				(font
@@
 		)
 		(property "Footprint" "Resistor_SMD:R_0603_1608Metric_Pad0.98x0.95mm_HandSolder"
-			(at 287.782 142.24 90)
+			(at 287.782 147.32 90)
 			(effects
 				(font
@@
 		)
 		(property "Datasheet" "~"
-			(at 289.56 142.24 0)
+			(at 289.56 147.32 0)
 			(effects
 				(font
@@
 		)
 		(property "Description" "Resistor"
-			(at 289.56 142.24 0)
+			(at 289.56 147.32 0)
 			(effects
 				(font
@@
 	)
 	(symbol
-		(lib_id "Device:R")
-		(at 323.85 146.05 90)
-		(unit 1)
-		(exclude_from_sim no)
-		(in_bom yes)
-		(on_board yes)
-		(dnp no)
-		(fields_autoplaced yes)
-		(property "Reference" "R3"
-			(at 323.85 139.7 90)
-			(effects
-				(font
-					(size 1.27 1.27)
-				)
-			)
-		)
-		(property "Value" "50"
-			(at 323.85 142.24 90)
-			(effects
-				(font
-					(size 1.27 1.27)
-				)
-			)
-		)
-		(property "Footprint" "Resistor_SMD:R_0805_2012Metric_Pad1.20x1.40mm_HandSolder"
-			(at 323.85 147.828 90)
-			(effects
-				(font
-					(size 1.27 1.27)
-				)
-				(hide yes)
-			)
-		)
-		(property "Datasheet" "~"
-			(at 323.85 146.05 0)
-			(effects
-				(font
-					(size 1.27 1.27)
-				)
-				(hide yes)
-			)
-		)
-		(property "Description" "Resistor"
-			(at 323.85 146.05 0)
-			(effects
-				(font
-					(size 1.27 1.27)
-				)
-				(hide yes)
-			)
-		)
-		(pin "1"
-		)
-		(pin "2"
-		)
-		(instances
-			(project ""
-				(path "/09bbc44e-8029-468d-a6fc-2a31dfd55e08"
-					(reference "R3")
-					(unit 1)
-				)
-			)
-		)
-	)
-	(symbol
 		(lib_id "power:GND")
 		(at 339.09 182.88 180)
@@
 		(on_board yes)
 		(dnp no)
-		(fields_autoplaced yes)
 		(property "Reference" "#FLG05"
 			(at 355.6 125.095 0)
@@
 		)
 		(property "Value" "PWR_FLAG"
-			(at 355.6 128.27 0)
+			(at 358.394 127.508 0)
 			(effects
 				(font
